File: Hardware/minisumo3-arreglo-smd/minisumo.kicad_sch (KiCad schematic)
At the start: 17 parts, among them J1 batterly, J2 hc-sr05, J3 sensor, M1 Motor_DC, M2 Motor_DC, SW1 SW_DPST_x2, U1 L293D, U2 L7805

Commit message: Add files via upload
Parts:
- U2: footprint componentes. pretty(huellas)_mod:TO-220-2 -> Package_TO_SOT_SMD:TO-263-3_TabPin2
Changed lines of the file:
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@@
 			)
 		)
-		(property "Footprint" "componentes. pretty(huellas)_mod:TO-220-2"
+		(property "Footprint" "Package_TO_SOT_SMD:TO-263-3_TabPin2"
 			(at 244.221 134.874 0)
 			(effects
